File: main.sch (EAGLE design)
At the start: 56 parts, among them CON1 451000, CON1_ 451000, CON2 451000, CON2_ 451000, IC1 MEGA8-AI, IC2 MC78M05ABDT, Q1 16MHz

Commit message: adding images of the current version
Parts:
- IC1: value MEGA8-AI -> ATMega88PA
Other:
- moved on the sheet: C6, C7, IC2, JP1, SV1, TP1, TP19, TP2, TP20

Commit message: Optokoppler für Daymode => Optokoppler für Datenleitung
Connections:
- net DOOR_DAYMODE renamed DOOR_DATA
- net DOOR_DAYMODE_+ renamed DOOR_DATA_+
- net DOOR_DAYMODE_- renamed DOOR_DATA_-
- net _DOOR_DAYMODE renamed _DOOR_DATA
Changed lines of the file:
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@@
-</segment>
-</net>
-<net name="DOOR_DAYMODE" class="0">
-<segment>
-<pinref part="IC1" gate="G$1" pin="PC2(ADC2)"/>
-<wire x1="121.92" y1="101.6" x2="124.46" y2="101.6" width="0.1524" layer="91"/>
-<label x="124.46" y="101.6" size="1.778" layer="95"/>
-</segment>
-<segment>
-<wire x1="160.02" y1="86.36" x2="162.56" y2="86.36" width="0.1524" layer="91"/>
-<pinref part="CON2" gate="G$1" pin="3"/>
-<label x="160.02" y="86.36" size="1.778" layer="95" rot="R180"/>
 </segment>
 </net>
@@
 </segment>
 </net>
-<net name="DOOR_DAYMODE_+" class="0">
+<net name="DOOR_DATA_+" class="0">
 <segment>
 <wire x1="276.86" y1="76.2" x2="274.32" y2="76.2" width="0.1524" layer="91"/>
@@
 </segment>
 </net>
-<net name="DOOR_DAYMODE_-" class="0">
+<net name="DOOR_DATA_-" class="0">
 <segment>
 <wire x1="276.86" y1="71.12" x2="274.32" y2="71.12" width="0.1524" layer="91"/>
@@
 </segment>
 </net>
-<net name="_DOOR_DAYMODE" class="0">
-<segment>
-<pinref part="R4" gate="G$1" pin="2"/>
-<wire x1="241.3" y1="71.12" x2="238.76" y2="71.12" width="0.1524" layer="91"/>
-<label x="238.76" y="71.12" size="1.778" layer="95" rot="R180"/>
-</segment>
-<segment>
-<wire x1="198.12" y1="86.36" x2="200.66" y2="86.36" width="0.1524" layer="91"/>
-<pinref part="CON2_" gate="G$1" pin="3"/>
-<label x="200.66" y="86.36" size="1.778" layer="95"/>
-</segment>
-</net>
 <net name="_DOOR_OPEN" class="0">
 <segment>
@@
 </segment>
 </net>
+<net name="DOOR_DATA" class="0">
+<segment>
+<pinref part="IC1" gate="G$1" pin="PC2(ADC2)"/>
+<wire x1="121.92" y1="101.6" x2="124.46" y2="101.6" width="0.1524" layer="91"/>
+<label x="124.46" y="101.6" size="1.778" layer="95"/>
+</segment>
+<segment>
+<wire x1="160.02" y1="86.36" x2="162.56" y2="86.36" width="0.1524" layer="91"/>
+<pinref part="CON2" gate="G$1" pin="3"/>
+<label x="160.02" y="86.36" size="1.778" layer="95" rot="R180"/>
+</segment>
+</net>
+<net name="_DOOR_DATA" class="0">
+<segment>
+<wire x1="198.12" y1="86.36" x2="200.66" y2="86.36" width="0.1524" layer="91"/>
+<pinref part="CON2_" gate="G$1" pin="3"/>
+<label x="200.66" y="86.36" size="1.778" layer="95"/>
+</segment>
+<segment>
+<pinref part="R4" gate="G$1" pin="2"/>
+<wire x1="241.3" y1="71.12" x2="238.76" y2="71.12" width="0.1524" layer="91"/>
+<label x="238.76" y="71.12" size="1.778" layer="95" rot="R180"/>
+</segment>
+</net>
